File: hardware/radioactivity-detector.sch (KiCad schematic (older format))
At the start: 21 parts, among them J1 Conn_01x02, J2 Conn_01x02, U1 OPA333xxD, U2 OPA333xxD

Commit message: fixed missing libraries
Parts:
- C1, C2, C3, C4, C5, C6, C7: symbol C -> Device:C
- C8: symbol CP -> Device:CP
- D1: symbol D_Photo -> Device:D_Photo
- J1, J2: symbol Conn_01x02 -> Connector:Conn_01x02_Female
- L1: symbol L_Core_Ferrite -> Device:L_Core_Ferrite
- R1, R2, R3, R4, R5, R6, R7: symbol R -> Device:R
- U1, U2: symbol OPA333xxD -> Amplifier_Operational:OPA330xxD
Changed lines of the file:
@@
 EESchema Schematic File Version 4
-LIBS:power
-LIBS:device
-LIBS:switches
-LIBS:relays
-LIBS:motors
-LIBS:transistors
-LIBS:conn
-LIBS:linear
-LIBS:regul
-LIBS:74xx
-LIBS:cmos4000
-LIBS:adc-dac
-LIBS:memory
-LIBS:xilinx
-LIBS:microcontrollers
-LIBS:dsp
-LIBS:microchip
-LIBS:analog_switches
-LIBS:motorola
-LIBS:texas
-LIBS:intel
-LIBS:audio
-LIBS:interface
-LIBS:digital-audio
-LIBS:philips
-LIBS:display
-LIBS:cypress
-LIBS:siliconi
-LIBS:opto
-LIBS:atmel
-LIBS:contrib
-LIBS:valves
 LIBS:radioactivity-detector-cache
 EELAYER 26 0
@@
 $EndDescr
 $Comp
-L D_Photo D1
+L Device:D_Photo D1
 U 1 1 5A537622
 P 6050 3950
@@
 $EndComp
 $Comp
-L GND #PWR01
+L power:GND #PWR01
 U 1 1 5A5376C9
 P 5750 4150
@@
 $EndComp
 $Comp
-L R R3
+L Device:R R3
 U 1 1 5A537870
 P 6700 3250
@@
 $EndComp
 $Comp
-L R R2
+L Device:R R2
 U 1 1 5A537971
 P 5750 3850
@@
 $EndComp
 $Comp
-L R R1
+L Device:R R1
 U 1 1 5A5379A2
 P 5750 3300
@@
 $EndComp
 $Comp
-L C C1
+L Device:C C1
 U 1 1 5A5379D1
 P 5450 3850
@@
 $EndComp
 $Comp
-L C C3
+L Device:C C3
 U 1 1 5A537AAB
 P 6700 2950
@@
 $EndComp
 $Comp
-L GND #PWR02
+L power:GND #PWR02
 U 1 1 5A537E00
 P 5450 4150
@@
 $EndComp
 $Comp
-L GND #PWR03
+L power:GND #PWR03
 U 1 1 5A5381A8
 P 6500 4150
@@
 $EndComp
 $Comp
-L C C2
+L Device:C C2
 U 1 1 5A538230
 P 7250 2850
@@
 $EndComp
 $Comp
-L GND #PWR04
+L power:GND #PWR04
 U 1 1 5A53840E
 P 7250 3050
@@
 $EndComp
 $Comp
-L Conn_01x02 J1
+L Connector:Conn_01x02_Female J1
 U 1 1 5A538563
 P 9950 3500
@@
 $EndComp
 $Comp
-L GND #PWR05
+L power:GND #PWR05
 U 1 1 5A5385ED
 P 9700 4150
@@
 $EndComp
 $Comp
-L C C5
+L Device:C C5
 U 1 1 5A54AF26
 P 7300 3600
@@
 $EndComp
 $Comp
-L R R5
+L Device:R R5
 U 1 1 5A54AF76
 P 7650 3600
@@
 $EndComp
 $Comp
-L R R6
+L Device:R R6
 U 1 1 5A54AFD7
 P 8750 3900
@@
 $EndComp
 $Comp
-L GND #PWR06
+L power:GND #PWR06
 U 1 1 5A54B1A7
 P 8500 4150
@@
 $EndComp
 $Comp
-L GND #PWR07
+L power:GND #PWR07
 U 1 1 5A54BDCB
 P 6050 4150
@@
 $EndComp
 $Comp
-L Conn_01x02 J2
+L Connector:Conn_01x02_Female J2
 U 1 1 5A54DDE0
 P 9950 2550
@@
 $EndComp
 $Comp
-L GND #PWR08
+L power:GND #PWR08
 U 1 1 5A54DE86
 P 9300 4150
@@
 $EndComp
 $Comp
-L L_Core_Ferrite L1
+L Device:L_Core_Ferrite L1
 U 1 1 5A54DEAF
 P 9300 2550
@@
 $EndComp
 $Comp
-L OPA333xxD U1
+L Amplifier_Operational:OPA330xxD U1
 U 1 1 5A54E9B2
 P 6600 3600
@@
 $EndComp
 $Comp
-L OPA333xxD U2
+L Amplifier_Operational:OPA330xxD U2
 U 1 1 5A54EB63
 P 8600 3500
@@
 $EndComp
 $Comp
-L R R4
+L Device:R R4
 U 1 1 5A54F51F
 P 8100 3150
@@
 $EndComp
 $Comp
-L R R7
+L Device:R R7
 U 1 1 5A54F5CD
 P 8100 3900
@@
 $EndComp
 $Comp
-L C C4
+L Device:C C4
 U 1 1 5A54F62E
 P 7800 3950
@@
 $EndComp
 $Comp
-L GND #PWR09
+L power:GND #PWR09
 U 1 1 5A54F69A
 P 7800 4150
@@
 $EndComp
 $Comp
-L GND #PWR010
+L power:GND #PWR010
 U 1 1 5A54F6DB
 P 8100 4150
@@
 	6500 2550 6500 2650
 $Comp
-L C C6
+L Device:C C6
 U 1 1 5A550718
 P 8750 2850
@@
 $EndComp
 $Comp
-L GND #PWR011
+L power:GND #PWR011
 U 1 1 5A55076B
 P 8750 3050
@@
 Connection ~ 8500 2650
 $Comp
-L C C7
+L Device:C C7
 U 1 1 5A550D62
 P 9050 2850
@@
 $EndComp
 $Comp
-L CP C8
+L Device:CP C8
 U 1 1 5A550DF6
 P 9550 2850
@@
 Connection ~ 9050 2550
 $Comp
-L GND #PWR012
+L power:GND #PWR012
 U 1 1 5A5510FD
 P 9050 4150
@@
 $EndComp
 $Comp
-L GND #PWR013
+L power:GND #PWR013
 U 1 1 5A551147
 P 9550 4150

Commit message: initial versionwq
Parts:
- removed J1, J2: Conn_01x02, Pin_Headers:Pin_Header_Straight_2x01_Pitch2.54mm, symbol Connector:Conn_01x02_Female
- removed U1, U2: OPA333xxD, Housings_SOIC:SO-8_5.3x6.2mm_Pitch1.27mm, symbol Amplifier_Operational:OPA330xxD
- added BT1, BT2, BT3, BT4: 12V, SemiconductorRadioactivityDetector:A23Single, symbol Device:Battery_Cell
- added C10: 10p, Capacitors_SMD:C_0805_HandSoldering, symbol Device:C
- added C11, C12, C4: 100n, Capacitors_SMD:C_0805_HandSoldering, symbol Device:C
- added D1, D2: D_Photo, Diodes_THT:D_DO-35_SOD27_P5.08mm_Vertical_KathodeUp, symbol Device:D_Photo
- added H1, H2, H3: MountingHole_Pad, Mounting_Holes:MountingHole_3.5mm_Pad, symbol Mechanical:MountingHole_Pad
- added J1: power, Connector_PinHeader_2.54mm:PinHeader_1x02_P2.54mm_Vertical, symbol Connector:Conn_01x02_Male
- added J2, J3: Conn_Coaxial, Connectors:BNC, symbol Connector:Conn_Coaxial
- added R10, R11, R12, R13, R9: 10k, Resistors_SMD:R_0805_HandSoldering, symbol Device:R
- added R3: 560k, Resistors_SMD:R_0805_HandSoldering, symbol Device:R
- added RV1: R_POT_TRIM, Potentiometers:Potentiometer_Trimmer_Bourns_3296W, symbol Device:R_POT_TRIM
- added U1, U2: OPA333xxD, Housings_SOIC:SOIC-8_3.9x4.9mm_Pitch1.27mm, symbol Amplifier_Operational:OPA333xxD
- added U4: LM358_DFN, Housings_SOIC:SOIC-8_3.9x4.9mm_Pitch1.27mm, symbol Amplifier_Operational:LM358_DFN
- C1: renamed from C8; value CP -> 100u
- C2: renamed from C7; footprint Capacitors_SMD:C_1206 -> Capacitors_SMD:C_0805_HandSoldering
- C3: renamed from C1; footprint Capacitors_SMD:C_1206 -> Capacitors_SMD:C_0805_HandSoldering
- C5: renamed from C2; footprint Capacitors_SMD:C_1206 -> Capacitors_SMD:C_0805_HandSoldering
- C6: renamed from C3; footprint Capacitors_SMD:C_1206 -> Capacitors_SMD:C_0805_HandSoldering
- C7: renamed from C5; footprint Capacitors_THT:C_Disc_D4.3mm_W1.9mm_P5.00mm -> Capacitors_SMD:C_0805_HandSoldering
- C8: renamed from C4; footprint Capacitors_SMD:C_1206 -> Capacitors_SMD:C_0805_HandSoldering
- C9: renamed from C6; footprint Capacitors_SMD:C_1206 -> Capacitors_SMD:C_0805_HandSoldering
- D3: renamed from D1; footprint Opto-Devices:PhotoDiode_BPW82 -> Diodes_THT:D_DO-35_SOD27_P5.08mm_Vertical_KathodeUp
- R1: value 1k -> 10k; footprint Resistors_THT:R_Axial_DIN0204_L3.6mm_D1.6mm_P7.62mm_Horizontal -> Resistors_SMD:R_0805_HandSoldering
- R2, R7: value 1k -> 10k; footprint Resistors_SMD:R_1206 -> Resistors_SMD:R_0805_HandSoldering
- R4: renamed from R3; value 10M -> 560k; footprint Resistors_SMD:R_MiniMELF_MMA-0204 -> Resistors_SMD:R_0805_HandSoldering
- R5: footprint Resistors_SMD:R_1206 -> Resistors_SMD:R_0805_HandSoldering
- R6: renamed from R4; value 1k -> 10k; footprint Resistors_SMD:R_1206 -> Resistors_THT:R_Axial_DIN0207_L6.3mm_D2.5mm_P10.16mm_Horizontal
- R8: renamed from R6; footprint Resistors_SMD:R_1206 -> Resistors_SMD:R_0805_HandSoldering
Connections:
- net GND: now also C5.1, C9.1, BT4.1 (+), C11.2, C4.1, H1.1, H2.1, H3.1, J1.2 (Pin_2), J2.2 (Ext), J3.2 (Ext), R11.2, R9.2, U1.4 (V-), U2.4 (V-), U4.4 (V-), U4.9 (PAD); no longer C5.2, C9.2, D3.2 (A)
- net at C6.2, R4.1: now also R3.2; no longer D3.1 (K)
- net at C6.1, C7.2, R4.2: now also U1.6
- net at C3.1, R1.2, R2.1: now also U1.3 (+)
- net at C2.1, L1.1, R1.1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: now also C5.2, C9.2, C11.1, R10.1, U1.7 (V+), U2.7 (V+), U4.8 (V+); no longer C5.1, C9.1
- net at R8.2: now also C10.1, U2.6, U4.3 (+), U4.5 (+)
- net at R5.2, R8.1: now also C10.2, U2.2 (-)
- net at C1.1, L1.2: now also J1.1 (Pin_1)
- net at C8.1, R6.2, R7.1: now also U2.3 (+)
- new net: D1.1 (K), D2.1 (K), D3.1 (K), R3.1, U1.2 (-)
- new net: BT1.2 (-), C4.2, D1.2 (A), D2.2 (A), D3.2 (A)
- new net: BT3.1 (+), BT4.2 (-)
- new net: BT2.1 (+), BT3.2 (-)
- new net: BT1.1 (+), BT2.2 (-)
- new net: C12.1, J2.1 (In), R9.1
- new net: C12.2, U4.1, U4.2 (-)
- new net: R12.1, R13.2, U4.6 (-)
- new net: J3.1 (In), R13.1, U4.7
- new net: R11.1, RV1.3
- new net: R10.2, RV1.1
- new net: R12.2, RV1.2
Other:
- note added: "amplifier"
- note added: "input"
- note added: "output"
- note added: "photodiode bias"
- note added: "power supply"
- moved on the sheet: C1, C2, C3, C5, C6, C7, C8, C9, D3, L1, R1, R2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
