File: hardware/radioactivity-detector.sch (KiCad schematic (older format))
At the start: 38 parts, among them J1 power, J2 Conn_Coaxial, U1 OPA333xxD, U2 OPA333xxD, U3 OPA333xxD

Commit message: last touch before sending to pcb factory
Parts:
- removed H4: MountingHole_Pad, Mounting_Holes:MountingHole_3.5mm_Pad, symbol Mechanical:MountingHole_Pad
- removed U3: OPA333xxD, Housings_SOIC:SOIC-8_3.9x4.9mm_Pitch1.27mm, symbol Amplifier_Operational:OPA333xxD
- added J3: Conn_Coaxial, Connectors:BNC, symbol Connector:Conn_Coaxial
- added R10, R11, R12, R13: 10k, Resistors_SMD:R_0805_HandSoldering, symbol Device:R
- added RV1: R_POT_TRIM, Potentiometers:Potentiometer_Trimmer_Bourns_3296W, symbol Device:R_POT_TRIM
- added U4: LM358_DFN, Housings_SOIC:SOIC-8_3.9x4.9mm_Pitch1.27mm, symbol Amplifier_Operational:LM358_DFN
- C10: value 1p -> 10p
- J2: footprint Connectors:PINHEAD1-2 -> Connectors:BNC
Connections:
- net GND: now also C11.2, J3.2 (Ext), R11.2, U4.4 (V-), U4.9 (PAD); no longer C11.1
- net at C2.1, C5.2, C9.2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: now also C11.1, R10.1, U4.8 (V+); no longer C11.2
- net at C10.1, R8.2, U2.6: now also U4.3 (+), U4.5 (+)
- net at C12.2: now also U4.1, U4.2 (-)
- new net: R12.1, R13.2, U4.6 (-)
- new net: J3.1 (In), R13.1, U4.7
- new net: R11.1, RV1.3
- new net: R10.2, RV1.1
- new net: R12.2, RV1.2
Other:
- moved on the sheet: C1, C11, C12, C2, C3, D1, D2, D3, H1, H2, H3, J2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
