File: hardware/radioactivity-detector.kicad_pcb (KiCad board)
At the start: 2 copper layers, 21 parts, among them J1 Conn_01x02, J2 Conn_01x02, U1 OPA333xxD, U2 OPA333xxD

Commit message: pcb fixes before sending to factory
Parts:
- moved C8 34.0 mm to (137.1, 103.7), turned to 90 degrees
- moved R6 30.5 mm to (141.4, 99.3)
- moved J1 30.0 mm to (146.0, 99.9)
- moved L1 30.0 mm to (133.3, 103.7)
- moved C6 29.5 mm to (133.9, 98.0)
- moved D1 29.5 mm to (137.1, 73.4)
- moved R1 29.5 mm to (141.6, 86.5)
- moved R2 29.5 mm to (147.3, 76.7)
- moved R3 29.5 mm to (137.1, 79.1)
- moved R4 29.5 mm to (133.9, 92.9)
- moved R5 29.5 mm to (140.9, 89.1)
- moved U1 29.5 mm to (142.2, 79.1)
- moved U2 29.5 mm to (141.6, 94.2)
- moved C1 29.5 mm to (144.7, 72.7)
- moved C4 29.5 mm to (133.9, 88.5)
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Routing:
- net Net-(R5-Pad2): track 13.6 -> 12.7 mm
- net Net-(C2-Pad1): track 45.8 -> 46.5 mm
- net GND: vias 0 -> 21
- added copper zone on F.Cu, net GND
Other:
- board outline added: 24.1 x 40.6 mm

Commit message: final touch before ordering pcb
Parts:
- added ground connector: MountingHole_2.2mm_M2, Mounting_Holes:MountingHole_2.2mm_M2, F.Cu at (109.0, 91.0)
- moved J2 40.0 mm to (108.7, 82.5), turned to 270 degrees
- moved L1 36.3 mm to (111.2, 74.9), turned to 180 degrees
- moved C8 36.0 mm to (111.2, 78.7), turned to 0 degrees
- moved J1 33.3 mm to (115.0, 87.6), turned to 270 degrees
- moved R6 30.5 mm to (115.7, 83.0), turned to 270 degrees
- moved C2 29.3 mm to (119.7, 90.1), turned to 180 degrees
- moved C6 28.2 mm to (116.9, 75.5), turned to 270 degrees
- moved C7 24.6 mm to (119.5, 75.5), turned to 270 degrees
- moved U2 23.6 mm to (120.7, 83.2), turned to 270 degrees
- moved R4 21.1 mm to (122.0, 75.5), turned to 270 degrees
- moved C5 19.4 mm to (125.8, 86.6), turned to 315 degrees
- moved R5 16.5 mm to (125.8, 82.5), turned to 90 degrees
- moved C4 15.5 mm to (126.5, 74.9), turned to 0 degrees
- moved R2 15.1 mm to (138.2, 88.9), turned to 0 degrees
- moved R7 14.9 mm to (126.5, 77.4), turned to 0 degrees
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Routing:
- net GND: track 0.00 -> 94.6 mm, vias 21 -> 11
- net Net-(C2-Pad1): track 46.5 -> 48.3 mm
- net Net-(C3-Pad2): track 13.2 -> 12.3 mm
Other:
- board size 24.1 x 40.6 mm -> 42.5 x 25 mm
- net class Default: via_dia 0.6 -> 1.3; via_drill 0.4 -> 0.6
- net class low signal removed
- board text added: "Semiconductor Radioactivity Sensor"
- board text added: "rev3.0"

Commit message: initial versionwq
Parts:
- removed ground connector: MountingHole_2.2mm_M2, Mounting_Holes:MountingHole_2.2mm_M2
- added BT1: 12V, SemiconductorRadioactivityDetector:A23Single, F.Cu at (152.4, 109.9)
- added BT2: 12V, SemiconductorRadioactivityDetector:A23Single, F.Cu at (151.1, 79.4)
- added BT3: 12V, SemiconductorRadioactivityDetector:A23Single, F.Cu at (153.0, 109.2)
- added BT4: 12V, SemiconductorRadioactivityDetector:A23Single, F.Cu at (178.4, 74.3)
- added C10: 1p, Capacitors_SMD:C_0805_HandSoldering, F.Cu at (209.6, 103.5)
- added C11: 100n, Capacitors_SMD:C_0805_HandSoldering, F.Cu at (218.4, 95.9)
- added C12: 100n, Capacitors_SMD:C_0805_HandSoldering, F.Cu at (222.2, 102.8)
- added C9: 100n, Capacitors_SMD:C_0805_HandSoldering, F.Cu at (213.4, 97.2)
- added D2: D_Photo, Diodes_THT:D_DO-35_SOD27_P5.08mm_Vertical_KathodeUp, B.Cu at (185.0, 98.7)
- added D3: D_Photo, Diodes_THT:D_DO-35_SOD27_P5.08mm_Vertical_KathodeUp, B.Cu at (185.0, 95.0)
- added H1: MountingHole_Pad, Mounting_Holes:MountingHole_3.5mm_Pad, F.Cu at (145.0, 75.0)
- added H2: MountingHole_Pad, Mounting_Holes:MountingHole_3.5mm_Pad, F.Cu at (145.0, 120.0)
- added H3: MountingHole_Pad, Mounting_Holes:MountingHole_3.5mm_Pad, F.Cu at (215.0, 75.0)
- added H4: MountingHole_Pad, Mounting_Holes:MountingHole_3.5mm_Pad, F.Cu at (215.0, 120.0)
- added R8: 1M, Resistors_SMD:R_0805_HandSoldering, F.Cu at (209.6, 106.0)
- added R9: 10k, Resistors_SMD:R_0805_HandSoldering, F.Cu at (220.3, 108.0)
- added U3: OPA333xxD, Housings_SOIC:SOIC-8_3.9x4.9mm_Pitch1.27mm, F.Cu at (217.8, 101.0)
- C1: value 100n -> 100u; footprint Capacitors_SMD:C_1206 -> Capacitors_Tantalum_SMD:CP_Tantalum_Case-A_EIA-3216-18_Hand; moved to F.Cu
- C2, C4: footprint Capacitors_SMD:C_1206 -> Capacitors_SMD:C_0805_HandSoldering; moved to F.Cu
- C3: value 2p -> 100n; footprint Capacitors_SMD:C_1206 -> Capacitors_SMD:C_0805_HandSoldering; moved to F.Cu
- C5: value 1n -> 100n; footprint Capacitors_THT:C_Disc_D4.3mm_W1.9mm_P5.00mm -> Capacitors_SMD:C_0805_HandSoldering
- C6: value 100n -> 2p; footprint Capacitors_SMD:C_1206 -> Capacitors_SMD:C_0805_HandSoldering; moved to F.Cu
- C7: value 100n -> 1n; footprint Capacitors_SMD:C_1206 -> Capacitors_SMD:C_0805_HandSoldering; moved to F.Cu
- C8: value CP -> 100n; footprint Capacitors_Tantalum_SMD:CP_Tantalum_Case-A_EIA-3216-18_Hand -> Capacitors_SMD:C_0805_HandSoldering; moved to F.Cu
- D1: footprint Opto-Devices:PhotoDiode_BPW82 -> Diodes_THT:D_DO-35_SOD27_P5.08mm_Vertical_KathodeUp; moved to B.Cu
- J1: value Conn_01x02 -> power; footprint Pin_Headers:Pin_Header_Straight_2x01_Pitch2.54mm -> Connector_PinHeader_2.54mm:PinHeader_1x02_P2.54mm_Vertical; moved to F.Cu
- J2: value Conn_01x02 -> Conn_Coaxial; footprint Pin_Headers:Pin_Header_Straight_2x01_Pitch2.54mm -> Connectors:PINHEAD1-2; moved to F.Cu
- L1: moved to F.Cu
- R1: value 1k -> 10k; footprint Resistors_THT:R_Axial_DIN0204_L3.6mm_D1.6mm_P7.62mm_Horizontal -> Resistors_SMD:R_0805_HandSoldering
- R2, R7: value 1k -> 10k; footprint Resistors_SMD:R_1206 -> Resistors_SMD:R_0805_HandSoldering; moved to F.Cu
- R3: value 10M -> 560k; footprint Resistors_SMD:R_MiniMELF_MMA-0204 -> Resistors_SMD:R_0805_HandSoldering; moved to F.Cu
- R4: value 1k -> 560k; footprint Resistors_SMD:R_1206 -> Resistors_SMD:R_0805_HandSoldering; moved to F.Cu
- R5: footprint Resistors_SMD:R_1206 -> Resistors_SMD:R_0805_HandSoldering; moved to F.Cu
- R6: value 1M -> 10k; footprint Resistors_SMD:R_1206 -> Resistors_THT:R_Axial_DIN0207_L6.3mm_D2.5mm_P10.16mm_Horizontal
- U1, U2: footprint Housings_SOIC:SO-8_5.3x6.2mm_Pitch1.27mm -> Housings_SOIC:SOIC-8_3.9x4.9mm_Pitch1.27mm; moved to F.Cu
- moved J2 113.9 mm to (219.1, 110.5)
- moved J1 106.0 mm to (221.0, 88.3), turned to 180 degrees
- moved L1 103.9 mm to (214.0, 90.2), turned to 90 degrees
- moved C2 99.4 mm to (219.1, 92.7), turned to 0 degrees
- moved C8 94.2 mm to (201.9, 104.1), turned to 180 degrees
- moved U2 89.1 mm to (208.3, 99.7), turned to 0 degrees
- moved R6 88.6 mm to (203.2, 96.5)
- moved R7 84.0 mm to (205.7, 105.3), turned to 270 degrees
- moved C7 83.1 mm to (198.8, 100.3), turned to 90 degrees
- moved C6 80.1 mm to (191.8, 104.1), turned to 180 degrees
- moved R5 77.5 mm to (201.3, 100.3)
- moved C1 75.6 mm to (217.8, 85.7), turned to 90 degrees
- moved C5 74.7 mm to (200.0, 95.4), turned to 225 degrees
- moved R4 74.5 mm to (191.8, 101.6), turned to 0 degrees
- moved R1 69.1 mm to (196.8, 93.3), turned to 180 degrees
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Connections:
- C2 pad 1: Net-(C2-Pad1) -> Net-(C11-Pad2)
- C3 pad 2: Net-(C3-Pad2) -> GND
- C4 pad 1: Net-(C4-Pad1) -> GND
- C4 pad 2: GND -> Net-(BT1-Pad2)
- C5 pad 1: Net-(C5-Pad1) -> GND
- C5 pad 2: Net-(C3-Pad1) -> Net-(C11-Pad2)
- C6 pad 1: Net-(C2-Pad1) -> Net-(C6-Pad1)
- C6 pad 2: GND -> Net-(C6-Pad2)
- C7 pad 1: Net-(C2-Pad1) -> Net-(C7-Pad1)
- C7 pad 2: GND -> Net-(C6-Pad1)
- D1 pad 1: Net-(C3-Pad2) -> Net-(D1-Pad1)
- D1 pad 2: GND -> Net-(BT1-Pad2)
- J1 pad 1: Net-(J1-Pad1) -> Net-(C1-Pad1)
- J2 pad 1: Net-(C8-Pad1) -> Net-(C12-Pad1)
- L1 pad 1: Net-(C2-Pad1) -> Net-(C11-Pad2)
- L1 pad 2: Net-(C8-Pad1) -> Net-(C1-Pad1)
- R1 pad 1: Net-(C2-Pad1) -> Net-(C11-Pad2)
- R1 pad 2: Net-(C1-Pad1) -> Net-(C3-Pad1)
- R2 pad 1: Net-(C1-Pad1) -> Net-(C3-Pad1)
- R3 pad 1: Net-(C3-Pad2) -> Net-(D1-Pad1)
- R3 pad 2: Net-(C3-Pad1) -> Net-(C6-Pad2)
- R4 pad 1: Net-(C2-Pad1) -> Net-(C6-Pad2)
- R4 pad 2: Net-(C4-Pad1) -> Net-(C6-Pad1)
- R5 pad 1: Net-(C5-Pad1) -> Net-(C7-Pad1)
- R5 pad 2: Net-(R5-Pad2) -> Net-(C10-Pad2)
- R6 pad 1: Net-(R5-Pad2) -> Net-(C11-Pad2)
- R6 pad 2: Net-(J1-Pad1) -> Net-(C8-Pad1)
- R7 pad 1: Net-(C4-Pad1) -> Net-(C8-Pad1)
- U1 pad 2: Net-(C3-Pad2) -> Net-(D1-Pad1)
- U1 pad 3: Net-(C1-Pad1) -> Net-(C3-Pad1)
- U1 pad 6: Net-(C3-Pad1) -> Net-(C6-Pad1)
- U1 pad 7: Net-(C2-Pad1) -> Net-(C11-Pad2)
- U2 pad 2: Net-(R5-Pad2) -> Net-(C10-Pad2)
- U2 pad 3: Net-(C4-Pad1) -> Net-(C8-Pad1)
- U2 pad 6: Net-(J1-Pad1) -> Net-(C10-Pad1)
- U2 pad 7: Net-(C2-Pad1) -> Net-(C11-Pad2)
Routing:
- net GND: track 94.6 -> 0.00 mm, vias 11 -> 0
- net Net-(C2-Pad1): track 48.3 -> 0.00 mm
- net Net-(C11-Pad2): track 0.00 -> 38.7 mm
- net Net-(BT1-Pad2): track 0.00 -> 23.8 mm
- net Net-(C10-Pad1): track 0.00 -> 19.3 mm
- net Net-(BT2-Pad1): track 0.00 -> 16.0 mm
- net Net-(D1-Pad1): track 0.00 -> 14.2 mm
- net Net-(BT3-Pad1): track 0.00 -> 13.4 mm
- net Net-(C10-Pad2): track 0.00 -> 13.3 mm
- net Net-(R5-Pad2): track 12.5 -> 0.00 mm
- net Net-(C3-Pad2): track 12.3 -> 0.00 mm
- net Net-(J1-Pad1): track 11.2 -> 0.00 mm
- net Net-(C6-Pad1): track 0.00 -> 11.1 mm
- net Net-(BT1-Pad1): track 0.00 -> 10.7 mm
- net Net-(C12-Pad2): track 0.00 -> 10.00 mm
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Other:
- board size 42.5 x 25 mm -> 90 x 55 mm
- board text added: "Semiconductor Radioactivity Detector"
- board text added: "rev3.1"
- board text removed: "Semiconductor Radioactivity Sensor"
- board text removed: "rev3.0"

Commit message: last touch before sending to pcb factory
Parts:
- removed H4: MountingHole_Pad, Mounting_Holes:MountingHole_3.5mm_Pad
- removed U3: OPA333xxD, Housings_SOIC:SOIC-8_3.9x4.9mm_Pitch1.27mm
- added J3: Conn_Coaxial, Connectors:BNC, F.Cu at (214.1, 102.4)
- added R10: 10k, Resistors_SMD:R_0805_HandSoldering, F.Cu at (216.2, 89.3)
- added R11: 10k, Resistors_SMD:R_0805_HandSoldering, F.Cu at (221.5, 103.8)
- added R12: 10k, Resistors_SMD:R_0805_HandSoldering, F.Cu at (216.1, 93.7)
- added R13: 10k, Resistors_SMD:R_0805_HandSoldering, F.Cu at (216.0, 96.8)
- added REF***: ESD-Logo_6.6x6mm_SilkScreen, Symbols:ESD-Logo_6.6x6mm_SilkScreen, F.Cu at (160.0, 80.8)
- added RV1: R_POT_TRIM, Potentiometers:Potentiometer_Trimmer_Bourns_3296W, F.Cu at (221.4, 93.3)
- added U4: LM358_DFN, Housings_SOIC:SOIC-8_3.9x4.9mm_Pitch1.27mm, F.Cu at (209.6, 93.3)
- C10: value 1p -> 10p
- J2: footprint Connectors:PINHEAD1-2 -> Connectors:BNC
- moved BT4 50.5 mm to (184.4, 124.5), turned to 180 degrees
- moved BT1 33.8 mm to (184.4, 99.1), turned to 180 degrees
- moved C4 27.6 mm to (173.2, 80.0)
- moved J2 24.9 mm to (195.6, 102.1), turned to 90 degrees
- moved D3 21.7 mm to (181.1, 73.7)
- moved R9 20.8 mm to (201.7, 98.6), turned to 315 degrees
- moved BT2 20.8 mm to (149.4, 100.1), turned to 0 degrees
- moved C12 20.6 mm to (203.2, 95.0), turned to 45 degrees
- moved D2 20.6 mm to (181.2, 78.5)
- moved D1 20.0 mm to (181.1, 82.9)
- moved BT3 18.2 mm to (135.6, 114.7)
- moved R2 18.0 mm to (187.8, 73.3)
- moved R3 18.0 mm to (184.0, 82.2)
- moved C10 18.0 mm to (205.6, 86.0)
- moved C5 18.0 mm to (196.1, 77.9)
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Connections:
- C11 pad 1: GND -> Net-(C11-Pad1)
- C11 pad 2: Net-(C11-Pad2) -> GND
- C2 pad 1: Net-(C11-Pad2) -> Net-(C11-Pad1)
- C5 pad 2: Net-(C11-Pad2) -> Net-(C11-Pad1)
- C9 pad 2: Net-(C11-Pad2) -> Net-(C11-Pad1)
- L1 pad 1: Net-(C11-Pad2) -> Net-(C11-Pad1)
- R1 pad 1: Net-(C11-Pad2) -> Net-(C11-Pad1)
- R6 pad 1: Net-(C11-Pad2) -> Net-(C11-Pad1)
- U1 pad 7: Net-(C11-Pad2) -> Net-(C11-Pad1)
- U2 pad 7: Net-(C11-Pad2) -> Net-(C11-Pad1)
Routing:
- net Net-(C11-Pad1): track 0.00 -> 40.8 mm
- net Net-(C11-Pad2): track 38.7 -> 0.00 mm
- net Net-(BT1-Pad2): track 23.8 -> 40.2 mm
- net Net-(J3-Pad1): track 0.00 -> 14.7 mm, vias 0 -> 2
- net Net-(BT2-Pad1): track 16.0 -> 28.4 mm
- net Net-(R12-Pad1): track 0.00 -> 6.75 mm
- net Net-(R10-Pad2): track 0.00 -> 6.14 mm
- net Net-(C12-Pad2): track 10.00 -> 4.62 mm
- net Net-(R12-Pad2): track 0.00 -> 4.86 mm
- net Net-(R11-Pad1): track 0.00 -> 4.04 mm
- net Net-(C10-Pad1): track 19.3 -> 23.2 mm
- net Net-(D1-Pad1): track 14.2 -> 16.8 mm
- net Net-(C12-Pad1): track 8.45 -> 10.8 mm
- net Net-(BT1-Pad1): track 10.7 -> 13.0 mm
- net GND: vias 0 -> 10
- removed copper zone on B.Cu, net GND
Other:
- outline, holes or cut-outs redrawn
- net class Default: via_dia 1.3 -> 1
- board text added: "Semiconductor Radioactivity Detector rev4.0"
- board text removed: "Semiconductor Radioactivity Detector"
- board text removed: "rev3.1"
