File: Hardware/SemiconductorRadioactivityDetector/SemiconductorRadioactivityDetector.kicad_sch (KiCad schematic)
At the start: 43 parts, among them J1 Conn_Coaxial, J2 Conn_Coaxial, J3 Conn_01x02_Pin, U1 OPA657U, U2 OPA656U, U3 LM358

Commit message: auxiliary board rev1.0
Parts:
- R4: value 1G -> 10G
Changed lines of the file:
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@@
 (kicad_sch
-	(version 20231120)
+	(version 20250114)
 	(generator "eeschema")
-	(generator_version "8.0")
+	(generator_version "9.0")
 	(paper "A4")
+	(text "input"
+		(exclude_from_sim no)
+		(at 105.41 58.42 0)
+		(effects
+			(font
+				(size 2.54 2.54)
+				(thickness 0.508)
+				(bold yes)
+			)
+			(justify left bottom)
+		)
+	)
+	(text "amplifier"
+		(exclude_from_sim no)
+		(at 160.02 58.42 0)
+		(effects
+			(font
+				(size 2.54 2.54)
+				(thickness 0.508)
+				(bold yes)
+			)
+			(justify left bottom)
+		)
+	)
+	(text "power supply"
+		(exclude_from_sim no)
+		(at 41.91 121.92 0)
+		(effects
+			(font
+				(size 2.54 2.54)
+				(thickness 0.508)
+				(bold yes)
+			)
+			(justify left bottom)
+		)
+	)
+	(text "output"
+		(exclude_from_sim no)
+		(at 218.44 58.42 0)
+		(effects
+			(font
+				(size 2.54 2.54)
+				(thickness 0.508)
+				(bold yes)
+			)
+			(justify left bottom)
+		)
+	)
+	(text "photodiode bias"
+		(exclude_from_sim no)
+		(at 121.92 133.35 0)
+		(effects
+			(font
+				(size 2.54 2.54)
+				(thickness 0.508)
+				(bold yes)
+			)
+			(justify left bottom)
+		)
+	)
 	(junction
 		(at 171.45 90.17)
@@
 		)
 	)
-	(text "input"
-		(exclude_from_sim no)
-		(at 105.41 58.42 0)
-		(effects
-			(font
-				(size 2.54 2.54)
-				(thickness 0.508)
-				(bold yes)
-			)
-			(justify left bottom)
-		)
-	)
-	(text "amplifier"
-		(exclude_from_sim no)
-		(at 160.02 58.42 0)
-		(effects
-			(font
-				(size 2.54 2.54)
-				(thickness 0.508)
-				(bold yes)
-			)
-			(justify left bottom)
-		)
-	)
-	(text "power supply"
-		(exclude_from_sim no)
-		(at 41.91 121.92 0)
-		(effects
-			(font
-				(size 2.54 2.54)
-				(thickness 0.508)
-				(bold yes)
-			)
-			(justify left bottom)
-		)
-	)
-	(text "output"
-		(exclude_from_sim no)
-		(at 218.44 58.42 0)
-		(effects
-			(font
-				(size 2.54 2.54)
-				(thickness 0.508)
-				(bold yes)
-			)
-			(justify left bottom)
-		)
-	)
-	(text "photodiode bias"
-		(exclude_from_sim no)
-		(at 121.92 133.35 0)
-		(effects
-			(font
-				(size 2.54 2.54)
-				(thickness 0.508)
-				(bold yes)
-			)
-			(justify left bottom)
-		)
-	)
 	(symbol
 		(lib_id "Device:D_Photo")
@@
 		(on_board yes)
 		(dnp no)
+		(fields_autoplaced yes)
 		(property "Reference" "R4"
 			(at 130.81 79.248 90)
@@
 			)
 		)
-		(property "Value" "1G"
+		(property "Value" "10G"
 			(at 130.81 81.28 90)
 			(effects
@@
 		(on_board yes)
 		(dnp no)
+		(fields_autoplaced yes)
 		(property "Reference" "R2"
-			(at 97.282 96.52 90)
+			(at 97.79 95.2499 0)
 			(effects
 				(font
 					(size 1.27 1.27)
 				)
+				(justify left)
 			)
 		)
 		(property "Value" "10k"
-			(at 95.25 96.52 90)
+			(at 97.79 97.7899 0)
 			(effects
 				(font
 					(size 1.27 1.27)
 				)
+				(justify left)
 			)
 		)
@@
 		(on_board yes)
 		(dnp no)
+		(fields_autoplaced yes)
 		(property "Reference" "R1"
-			(at 97.282 82.55 90)
+			(at 97.79 81.2799 0)
 			(effects
 				(font
 					(size 1.27 1.27)
 				)
+				(justify left)
 			)
 		)
 		(property "Value" "10k"
-			(at 95.25 82.55 90)
+			(at 97.79 83.8199 0)
 			(effects
 				(font
 					(size 1.27 1.27)
 				)
+				(justify left)
 			)
 		)
@@
 		)
 	)
+	(embedded_fonts no)
 )
