File: Hardware/SemiconductorRadioactivityDetector/SemiconductorRadioactivityDetector.kicad_pcb (KiCad board)
At the start: 2 copper layers, 90 x 55 mm, 43 parts, among them J1 Conn_Coaxial, J2 Conn_Coaxial, J3 Conn_01x02_Pin, U1 OPA333xxD, U2 OPA333xxD, U3 LM358

Commit message: auxiliary board rev2 + its 3d printed holder
Other:
- outline, holes or cut-outs redrawn
